File: PCB/quickpadPCM.kicad_pcb (KiCad board)
At the start: 2 copper layers, 92 x 59 mm, 10 parts, among them SW1 SW_Push, SW2 RotaryEncoder_Switch, SW3 SW_Push, SW4 SW_Push, SW5 SW_Push, SW6 SW_Push, SW7 SW_Push, SW8 SW_Push, SW9 SW_Push, U1 MOUDLE-SEEEDUINO-XIAO

Commit message: moved to br
Parts:
- moved SW2 27.4 mm to (69.0, 92.5)
- moved SW9 26.9 mm to (59.5, 70.9)
Routing:
- net Net-(U1-PB09_A7_D7_RX): track 78.7 -> 0.14 mm
- net Net-(U1-PB08_A6_D6_TX): track 53.4 -> 0.00 mm
- net Net-(U1-PA6_A10_D10_MOSI): track 107.8 -> 68.1 mm
- net Net-(U1-PA7_A8_D8_SCK): track 48.6 -> 18.2 mm
- net Net-(U1-PA11_A3_D3): track 52.6 -> 35.0 mm
- net Net-(U1-PA9_A5_D5_SCL): track 36.6 -> 50.1 mm
- net GND: track 175.6 -> 188.2 mm
- net Net-(U1-PA4_A1_D1): track 51.7 -> 50.8 mm
- net Net-(U1-PA5_A9_D9_MISO): track 72.0 -> 71.4 mm
- net Net-(U1-PA10_A2_D2): track 31.5 -> 30.9 mm

Commit message: finished wiring after moving encoder to a corner
Connections:
- SW2 pad A: Net-(U1-PA11_A3_D3) -> Net-(U1-GND)
- SW2 pad B: Net-(U1-PB08_A6_D6_TX) -> Net-(U1-3V3)
- SW2 pad S1: Net-(U1-PA9_A5_D5_SCL) -> Net-(U1-PA6_A10_D10_MOSI)
- SW3 pad 1: Net-(U1-PA6_A10_D10_MOSI) -> Net-(U1-5V)
- SW8 pad 1: Net-(U1-PA8_A4_D4_SDA) -> Net-(U1-PA11_A3_D3)
- SW9 pad 1: Net-(U1-PA7_A8_D8_SCK) -> Net-(U1-PA8_A4_D4_SDA)
- U1 pad 12: unconnected-(U1-3V3-Pad12) -> Net-(U1-3V3)
- U1 pad 13: unconnected-(U1-GND-Pad13) -> Net-(U1-GND)
- U1 pad 14: unconnected-(U1-5V-Pad14) -> Net-(U1-5V)
- U1 pad 6: Net-(U1-PA9_A5_D5_SCL) -> unconnected-(U1-PA9_A5_D5_SCL-Pad6)
- U1 pad 7: Net-(U1-PB08_A6_D6_TX) -> unconnected-(U1-PB08_A6_D6_TX-Pad7)
- U1 pad 9: Net-(U1-PA7_A8_D8_SCK) -> unconnected-(U1-PA7_A8_D8_SCK-Pad9)
Routing:
- net Net-(U1-5V): track 0.00 -> 104.7 mm
- net Net-(U1-GND): track 0.00 -> 82.6 mm
- net Net-(U1-PB09_A7_D7_RX): track 0.14 -> 78.7 mm
- net Net-(U1-3V3): track 0.00 -> 72.5 mm
- net Net-(U1-PA9_A5_D5_SCL): track 50.1 -> 0.00 mm
- net Net-(U1-PA8_A4_D4_SDA): track 22.8 -> 41.9 mm
- net Net-(U1-PA7_A8_D8_SCK): track 18.2 -> 0.00 mm
- net Net-(U1-PA6_A10_D10_MOSI): track 68.1 -> 53.1 mm
- net Net-(U1-PA11_A3_D3): track 35.0 -> 22.8 mm
- net unconnected-(U1-PA7_A8_D8_SCK-Pad9): track 0.00 -> 1.04 mm
Other:
- board size 92 x 59 mm -> 95.5 x 60 mm

Commit message: save
Parts:
- moved SW1 84.5 mm to (109.0, 101.5), turned to 180 degrees
- moved SW5 73.3 mm to (109.0, 63.6), turned to 180 degrees
- moved SW3 69.4 mm to (109.0, 82.6), turned to 180 degrees
- moved U1 65.9 mm to (42.1, 81.3), turned to 180 degrees
- moved SW4 58.2 mm to (90.0, 101.5), turned to 180 degrees
- moved SW6 50.1 mm to (71.0, 101.5), turned to 180 degrees
- moved SW7 40.2 mm to (90.0, 63.6), turned to 180 degrees
- moved SW2 33.5 mm to (80.5, 61.0), turned to 180 degrees
- moved SW9 32.6 mm to (90.0, 82.6), turned to 180 degrees
- moved SW8 13.9 mm to (71.0, 82.6), turned to 180 degrees
